Commit message: urdf-semidone

File: r_platform/urdf/r_platform_macro.urdf.xacro (robot description, xacro)
@@ -10,6 +10,6 @@
     				<mesh filename ="package://r_platform/CAD/robot-1.stl" />
     			</geometry>
-    			<material name ="LightGrey">
-        			<color rgba="0.83 0.83 0.83 1.0"/>
+    			<material name ="black">
+        		<color rgba="0.5 0.5 0.5 1.0"/>
         		</material>
     		</visual>
@@ -21,6 +21,6 @@
     				<mesh filename ="package://r_platform/CAD/CenaNova-1.stl" />
     			</geometry>
-    			<material name ="LightGrey">
-        			<color rgba="0.83 0.83 0.83 1.0"/>
+    			<material name ="blue">
+        			<color rgba="0 0.5 0.5 1.0"/>
         		</material>
     		</visual>
@@ -32,5 +32,5 @@
     				<mesh filename ="package://r_platform/CAD/CenaNovaLaser-1.stl" />
     			</geometry>
-    			<material name ="LightGrey">
+    			<material name ="blue">
         			<color rgba="0.83 0.83 0.83 1.0"/>
         		</material>
@@ -43,5 +43,5 @@
     				<mesh filename ="package://r_platform/CAD/Curva-1.stl" />
     			</geometry>
-    			<material name ="LightGrey">
+    			<material name ="blue">
         			<color rgba="0.83 0.83 0.83 1.0"/>
         		</material>
@@ -54,5 +54,5 @@
     				<mesh filename ="package://r_platform/CAD/Placa-Cima-1.stl" />
     			</geometry>
-    			<material name ="LightGrey">
+    			<material name ="blue">
         			<color rgba="0.83 0.83 0.83 1.0"/>
         		</material>
