Commit message: 1stage_DONE

File: r_platform/urdf/r_platform_macro.xacro (robot description, xacro)
@@ -131,5 +131,5 @@
             </collision>
         </link>
-        <joint name="base_Rwheel" type="continuous">
+        <joint name="base_Rwheel" type="fixed">
             <origin xyz="0.62 -0.03 0.5" rpy="0 0 0" />
             <parent link="plataform_base_link" />
@@ -159,5 +159,5 @@
             </collision>
         </link>
-        <joint name="base_Lwheel" type="continuous">
+        <joint name="base_Lwheel" type="fixed">
             <origin xyz="0.62 -0.03 -0.03" rpy="0 0 1.1753" />
             <parent link="plataform_base_link" />
