Commit message: interface+calibração

File: Bin-picking/bin_picking/urdf/binpicking_macro.xacro (robot description, xacro)
@@ -63,12 +63,12 @@
                 xyz="0.245525842462 0.115779043096 -0.017838428638"
                 rpy="-1.24022884812 1.5657875395 0.312412981998" /> -->
-             <!-- After Visions class X verry Bad  x: 0.330733  y: 0.190187 BEST  -->
+             <!-- J BEST  -->
+            <!-- <origin
+                xyz="0.242425842462 0.115779043096 -0.017838428638"
+                rpy="-1.24022884812 1.5657875395 0.312412981998" /> -->
+             <!-- TT 14-maio-2019-->
             <origin
-                xyz="0.242425842462 0.115779043096 -0.017838428638"
-                rpy="-1.24022884812 1.5657875395 0.312412981998" />
-             <!-- After Visions class X verry Bad  x: 0.3303 mas tambem pode ser 328.8  y: 0.190187 -->
-            <!-- <origin
-                xyz="0.242025842462 0.115779043096 -0.017838428638"
-                rpy="-1.24022884812 1.5657875395 0.312412981998" /> -->
+                xyz="0.261464612 0.124547681328 -0.0261357869128"
+                rpy="1.52288933699 1.55438293084 3.07729255495" />
         </xacro:kinect_camera>
     </xacro:macro>

File: Bin-picking/bin_picking/urdf/binpicking_sensor_macro.xacro (robot description, xacro)
@@ -5,6 +5,6 @@
         <link name="${prefix}base_link" />
         <joint name="${prefix}base_link-${prefix}optical_frame" type="fixed">
-            <origin xyz="0.0478 0.0166 -0.0636" rpy="0 0 0" />
-            <!-- <origin xyz="0.0478 0.0166 -0.0646" rpy="0 0 0" /> -->
+            <!-- <origin xyz="0.0478 0.0166 -0.0636" rpy="0 0 0" /> -->
+            <origin xyz="0.047 0.016 -0.0636" rpy="0 0 0" />
             <parent link="${prefix}base_link" />
             <child link="${prefix}optical_frame" />

File: robonuc_integration/urdf/robonuc_macro.xacro (robot description, xacro)
@@ -6,5 +6,5 @@
     <xacro:bin_picking prefix="" />
     <!-- include r_platform+sensores-->
-    <xacro:include filename="$(find r_platform)/urdf/r_platform_macro.xacro"/>
+    <xacro:include filename="$(find r_platform)/urdf/r_platform_and_hokuyo_macro.xacro"/>
     <xacro:r_platform prefix="" />
     <joint name="robot_base_link-Placa_cima" type="fixed">

Commit message: camera calib OK & launch for interface

File: Bin-picking/bin_picking/urdf/binpicking_macro.xacro (robot description, xacro)
@@ -11,56 +11,4 @@
         <xacro:bin_picking_manipulator prefix="${prefix}" />
         <xacro:kinect_camera name="camera" parent="${prefix}robot_link_4">
-             <!-- After Visions class X verry good x:0.330293 Y BAD y:0.199388    -->
-            <!-- <origin
-                xyz="0.247595042515 0.119885890773 -0.020976224609"
-                rpy="-1.16471837775 1.56523311718 0.4010175495" /> -->
-             <!-- After Visions class X verry good x:0.330293 Y BAD y:0.199388    -->
-            <!-- <origin
-                xyz="0.247469111314 0.121665921033 -0.0209441353601"
-                rpy="-1.73229551223 1.56538317963 -0.168783829812" /> -->
-             <!-- After Visions class X verry good x:0.334 Y BAD y:0.195    -->
-            <!-- <origin
-                xyz="0.246027243916 0.123698162921 -0.0217020720854"
-                rpy="-2.08465796645 1.56316258117 -0.51351285704" /> -->
-             <!-- After Visions class X verry Bad   x: 0.335595  y: 0.197092 -->
-            <!-- <origin
-                xyz="0.279701284349 0.120790055045 -0.0218256377425"
-                rpy="-1.45806785305 1.56396145711 0.108188416383" /> -->
-             <!-- After Visions class X verry Bad   x: 0.309  y: 0.194 -->
-            <!-- <origin
-                xyz="0.248302667803 0.116857146075 -0.0200601728922"
-                rpy="-0.344850120367 1.56341182063 1.20453906713" /> -->
-             <!-- After Visions class X verry Bad  x: 0.336117  y: 0.196357 -->
-            <!-- <origin
-                xyz="0.248185448612 0.125125454595 -0.0200843255582"
-                rpy="-2.38753667624 1.56620697644 -0.824028438096" /> -->
-             <!-- After Visions class X verry Bad  x: 0.337626  y: 0.187725 -->
-            <!-- <origin
-                xyz="0.250665005218 0.113460975328 -0.0160878898623"
-                rpy="0.300623743189 1.56621707328 1.83520171316" /> -->
-             <!-- After Visions class X verry Bad  x: 0.333275  y: 0.189395 -->
-            <!-- <origin
-                xyz="0.246027243916 0.114460975328 -0.0160878898623"
-                rpy="0.300623743189 1.56621707328 1.83520171316" /> -->
-             <!-- After Visions class X verry Bad x: 0.333779  y: 0.191524 -->
-            <!-- <origin
-                xyz="0.246027243916 0.114460975328 -0.0160878898623"
-                rpy="-0.5940411655 1.56143330405 0.976778156421" /> -->
-             <!-- After Visions class X verry Bad  x: 0.335904  y: 0.195349 -->
-            <!-- <origin
-                xyz="0.248036425169 0.11731055525 -0.0227873939643"
-                rpy="-0.888625605858 1.56465194539 0.663431270648" /> -->
-             <!-- After Visions class X verry Bad  x: 0.335904  y: 0.195349 -->
-            <!-- <origin
-                xyz="0.247753167311 0.117209715472 -0.0211379268936"
-                rpy="-0.5940411655 1.56143330405 0.976778156421" /> -->
-             <!-- After Visions class X verry Bad  x: 0.335904  y: 0.195349 -->
-            <!-- <origin
-                xyz="0.245902887069 0.122097650666 -0.0210615785857"
-                rpy="-1.94792098497 1.56412947012 -0.385098127041" /> -->
-             <!-- After Visions class X verry Bad  x: 0.33381  y: 0.190073 -->
-            <!-- <origin
-                xyz="0.245525842462 0.115779043096 -0.017838428638"
-                rpy="-1.24022884812 1.5657875395 0.312412981998" /> -->
              <!-- J BEST  -->
             <!-- <origin
@@ -68,7 +16,35 @@
                 rpy="-1.24022884812 1.5657875395 0.312412981998" /> -->
              <!-- TT 14-maio-2019-->
+            <!-- <origin
+                xyz="0.261464612 0.124547681328 -0.0261357869128"
+                rpy="1.52288933699 1.55438293084 3.07729255495" /> -->
+            <!-- TT 15-maio-2019 (com default intrinsec) Horrivel -->
+            <!-- <origin
+                xyz="0.275227080278 0.106485407928 -0.0247922882851"
+                rpy="-0.291826989842 1.4949234245 1.22820412985" /> -->
+            <!-- TT 16-maio-2019 (J intrinsecs) T1 (Best)-->
             <origin
-                xyz="0.261464612 0.124547681328 -0.0261357869128"
-                rpy="1.52288933699 1.55438293084 3.07729255495" />
+                xyz="0.254881746287 0.128927213047 -0.0237188254049"
+                rpy="2.03114796593 1.54366070438 -2.67392737672" />
+            <!-- TT 16-maio-2019 (J intrinsecs) T1 (á pata / good x y)-->
+            <!-- <origin
+                xyz="0.251881746287 0.125927213047 -0.0237188254049"
+                rpy="2.03114796593 1.54366070438 -2.67392737672" /> -->
+            <!-- TT 16-maio-2019 (J intrinsecs) T1 (á pata / GOOD mas afastado very bad! )-->
+            <!-- <origin
+                xyz="0.250081746287 0.124027213047 -0.0237188254049"
+                rpy="2.03114796593 1.54366070438 -2.67392737672" /> -->
+            <!-- TT 16-maio-2019 (J intrinsecs) T2 (Horrivel?)-->
+            <!-- <origin
+                xyz="0.275338115552 0.103474061974 -0.0163858909259"
+                rpy="0.348867591709 1.5462911626 1.9024420825" /> -->
+            <!-- TT 16-maio-2019 (J intrinsecs) T3 (muito má - horrivel) -->
+            <!-- <origin
+                xyz="0.289118892334 0.123446524013 -0.0230641291597"
+                rpy="1.63245885655 1.55214517793 -3.09749130672" /> -->
+            <!-- TT 16-maio-2019 (J intrinsecs) T4 ()-->
+            <!-- <origin
+                xyz="0.250061113358 0.121382628772 -0.0162125374077"
+                rpy="1.80615250348 1.55860488068 -2.93925623528" /> -->
         </xacro:kinect_camera>
     </xacro:macro>

File: Bin-picking/bin_picking/urdf/binpicking_sensor_macro.xacro (robot description, xacro)
@@ -6,5 +6,5 @@
         <joint name="${prefix}base_link-${prefix}optical_frame" type="fixed">
             <!-- <origin xyz="0.0478 0.0166 -0.0636" rpy="0 0 0" /> -->
-            <origin xyz="0.047 0.016 -0.0636" rpy="0 0 0" />
+            <origin xyz="0.0485 0.016 -0.0636" rpy="0 0 0" />
             <parent link="${prefix}base_link" />
             <child link="${prefix}optical_frame" />

Commit message: final_update

File: Bin-picking/bin_picking/urdf/binpicking_macro.xacro (robot description, xacro)
@@ -27,4 +27,12 @@
                 xyz="0.254881746287 0.128927213047 -0.0237188254049"
                 rpy="2.03114796593 1.54366070438 -2.67392737672" />
+		<!-- TT 10-junho-2019 (J intrinsecs) T1-->
+            <!-- <origin
+                xyz="0.234823726866 0.129533016016 0.0180443283311"
+                rpy="2.88805229371 1.53839584357 -1.81277150312" /> -->
+		<!-- TT 10-junho-2019 (J intrinsecs) T2-->
+            <!-- <origin
+                xyz="0.251945525019 0.11393756598 -0.0196092209476"
+                rpy="0.974144844099 1.55089696505 2.52009669515" /> -->
             <!-- TT 16-maio-2019 (J intrinsecs) T1 (á pata / good x y)-->
             <!-- <origin
